File: pcb/hhskb2.sch (KiCad schematic (older format))
At the start: 64 parts, among them SW00 SW_PUSH, SW01 SW_PUSH, SW02 SW_PUSH, SW03 SW_PUSH, SW04 SW_PUSH, SW05 SW_PUSH, SW10 SW_PUSH, SW11 SW_PUSH, SW12 SW_PUSH, SW13 SW_PUSH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

Commit message: 注文
Parts:
- removed D43: D, symbol D
- removed J?: 4pin_Jack, symbol 4pin_Jack
- removed R? (x2): R, symbol R
- removed SW43: SW_PUSH, symbol SW_PUSH
- added J1_right1, J2_left1: 4pin_Jack, MyFootprint:4pin_Jack, symbol 4pin_Jack
- added LED0, LED1, LED2: LED, LEDs:LED_D3.0mm, symbol LED
- added R0, R1, R2: R, Resistors_ThroughHole:R_Axial_DIN0207_L6.3mm_D2.5mm_P7.62mm_Horizontal, symbol R
- D0: renamed from D00; footprint (none) -> Diodes_ThroughHole:D_DO-41_SOD81_P7.62mm_Horizontal
- D1: renamed from D01; footprint (none) -> Diodes_ThroughHole:D_DO-41_SOD81_P7.62mm_Horizontal
- D10, D11, D12, D13, D14, D15, D20, D21, D22, D23, D24, D25, D30, D31, D32, D33, D34, D35, D40, D41, D42, D44, D45: footprint (none) -> Diodes_ThroughHole:D_DO-41_SOD81_P7.62mm_Horizontal
- D2: renamed from D02; footprint (none) -> Diodes_ThroughHole:D_DO-41_SOD81_P7.62mm_Horizontal
- D3: renamed from D03; footprint (none) -> Diodes_ThroughHole:D_DO-41_SOD81_P7.62mm_Horizontal
- D4: renamed from D04; footprint (none) -> Diodes_ThroughHole:D_DO-41_SOD81_P7.62mm_Horizontal
- D5: renamed from D05; footprint (none) -> Diodes_ThroughHole:D_DO-41_SOD81_P7.62mm_Horizontal
- SW0: renamed from SW00; footprint (none) -> MyFootprint:CHERRY_PLATE_100H
- SW1: renamed from SW01; footprint (none) -> MyFootprint:CHERRY_PLATE_100H
- SW10, SW11, SW12, SW13, SW14, SW15, SW20, SW21, SW22, SW23, SW24, SW25, SW30, SW31, SW32, SW33, SW34, SW35, SW42: footprint (none) -> MyFootprint:CHERRY_PLATE_100H
- SW2: renamed from SW02; footprint (none) -> MyFootprint:CHERRY_PLATE_100H
- SW3: renamed from SW03; footprint (none) -> MyFootprint:CHERRY_PLATE_100H
- SW4: renamed from SW04; footprint (none) -> MyFootprint:CHERRY_PLATE_100H
- SW40, SW41, SW44, SW45: footprint (none) -> MyFootprint:CHERRY_PLATE_125H
- SW5: renamed from SW05; footprint (none) -> MyFootprint:CHERRY_PLATE_100H
- U0: renamed from U?; footprint (none) -> arduino_micro_shield:ARDUINO_MICRO_SHIELD
Connections:
- net labels added: LED0, LED1, LED2
- wire segments 119 -> 128
- no-connect marks 16 -> 12
Other:
- note added: "COL INPUT_PULLUP Negative HIGH\n"
